File: tracks/A/MCX-A153_Shield_Template/MCX-A153_Shield_Template.kicad_pcb (KiCad board)
At the start: 2 copper layers, 91.4 x 54.6 mm, 13 parts, among them J1 Conn_02x08_Odd_Even, J2 Conn_02x10_Odd_Even, J3 Conn_02x08_Odd_Even, J4 Conn_02x06_Odd_Even

Commit message: -> Added labels to the schematics.
Parts:
- renumbered J4 to JJ4
Connections:
- J1 pad 1: unconnected-(J1-Pin_1-Pad1) -> /P1-7/GPIO
- J1 pad 10: unconnected-(J1-Pin_10-Pad10) -> /P2-5/GPIO
- J1 pad 12: unconnected-(J1-Pin_12-Pad12) -> /P3-12/PWM0
- J1 pad 14: unconnected-(J1-Pin_14-Pad14) -> /P3-13/PWM0
- J1 pad 16: unconnected-(J1-Pin_16-Pad16) -> /P3-1/GPIO
- J1 pad 2: unconnected-(J1-Pin_2-Pad2) -> /P1-4/RXD
- J1 pad 3: unconnected-(J1-Pin_3-Pad3) -> /P1-6/TRIG2
- J1 pad 4: unconnected-(J1-Pin_4-Pad4) -> /P1-5/TXD
- J1 pad 6: unconnected-(J1-Pin_6-Pad6) -> /P2-4/GPIO
- J1 pad 8: unconnected-(J1-Pin_8-Pad8) -> /P3-0/PWM0
- J2 pad 1: unconnected-(J2-Pin_1-Pad1) -> /P1-4/ADC0
- J2 pad 10: unconnected-(J2-Pin_10-Pad10) -> /P2-16/SDI1
- J2 pad 12: unconnected-(J2-Pin_12-Pad12) -> /P2-12/SCK1
- J2 pad 14: unconnected-(J2-Pin_14-Pad14) -> GND
- J2 pad 16: unconnected-(J2-Pin_16-Pad16) -> VDDA
- J2 pad 18: unconnected-(J2-Pin_18-Pad18) -> /P1-8/SDA0
- J2 pad 2: unconnected-(J2-Pin_2-Pad2) -> /P3-15/GPIO
- J2 pad 20: unconnected-(J2-Pin_20-Pad20) -> /P1-9/SCL0
- J2 pad 3: unconnected-(J2-Pin_3-Pad3) -> /P1-5/ADC0
- J2 pad 4: unconnected-(J2-Pin_4-Pad4) -> /P3-14/PWM0
- J2 pad 5: unconnected-(J2-Pin_5-Pad5) -> /P2-3/ADC0
- J2 pad 6: unconnected-(J2-Pin_6-Pad6) -> /P2-6/CSI1
- J2 pad 7: unconnected-(J2-Pin_7-Pad7) -> /P2-1/ADC0
- J2 pad 8: unconnected-(J2-Pin_8-Pad8) -> /P2-13/SDO1
- J2 pad 9: unconnected-(J2-Pin_9-Pad9) -> /P2-2/ADC0
- J3 pad 1: unconnected-(J3-Pin_1-Pad1) -> /P2-7/TRIG10
- J3 pad 10: unconnected-(J3-Pin_10-Pad10) -> /SYS-5V
- J3 pad 11: unconnected-(J3-Pin_11-Pad11) -> /P3-8/PWM0
- J3 pad 12: unconnected-(J3-Pin_12-Pad12) -> GND
- J3 pad 13: unconnected-(J3-Pin_13-Pad13) -> /P3-7/PWM0
- J3 pad 14: unconnected-(J3-Pin_14-Pad14) -> GND
- J3 pad 15: unconnected-(J3-Pin_15-Pad15) -> /P3-6/PWM0
- J3 pad 16: unconnected-(J3-Pin_16-Pad16) -> /5-9VIN
- J3 pad 3: unconnected-(J3-Pin_3-Pad3) -> /P3-31/TRIG5
- J3 pad 4: unconnected-(J3-Pin_4-Pad4) -> /VDD_BOARD
- J3 pad 5: unconnected-(J3-Pin_5-Pad5) -> /P3-11/PWM0
- J3 pad 6: unconnected-(J3-Pin_6-Pad6) -> /MCU_Reset
- J3 pad 7: unconnected-(J3-Pin_7-Pad7) -> /P3-10/PWM0
- J3 pad 8: unconnected-(J3-Pin_8-Pad8) -> /LDO_3v3
- J3 pad 9: unconnected-(J3-Pin_9-Pad9) -> /P3-9/PWM0
- JJ4 pad 10: unconnected-(JJ4-Pin_10-Pad10) -> /P3-31/ADC0
- JJ4 pad 11: unconnected-(JJ4-Pin_11-Pad11) -> /P3-29/GPIO
- JJ4 pad 12: unconnected-(JJ4-Pin_12-Pad12) -> /P3-30/ADC0
- JJ4 pad 2: unconnected-(JJ4-Pin_2-Pad2) -> /P1-10/ADC0
- JJ4 pad 4: unconnected-(JJ4-Pin_4-Pad4) -> /P1-12/ADC0
- JJ4 pad 6: unconnected-(JJ4-Pin_6-Pad6) -> /P1-13/ADC0
- JJ4 pad 8: unconnected-(JJ4-Pin_8-Pad8) -> /P2-0/ADC0
- JJ4 pad 9: unconnected-(JJ4-Pin_9-Pad9) -> /P1-11/GPIO
Routing:
- added copper zone on B.Cu, net GND
