File: tracks/A/Kicad/MCX-A153_Shield_Template.kicad_sch (KiCad schematic)
At the start: 8 parts, among them J1 Conn_02x08_Odd_Even, J2 Conn_02x10_Odd_Even, J3 Conn_02x08_Odd_Even

Commit message: minor tweaks before 1st release.  Added Altium version
Parts:
- renumbered JJ4 to J4
Connections:
- net LDO_3v3 renamed LDO-3v3
- net MCU_Reset renamed MCU-RESETb
- net P1-10/ADC0 renamed P1-10/ADC0-A8
- net P1-12/ADC0 renamed P1-12/ADC0-A10
- net P1-13/ADC0 renamed P1-13/ADC0-A11
- net P1-4/ADC0 renamed P1-4/ADC0-A20
- net P1-4/RXD renamed P1-4/UART2-RXD
- net P1-5/ADC0 renamed P1-5/ADC0-A21
- net P1-5/TXD renamed P1-5/UART2-TXD
- net P2-0/ADC0 renamed P2-0/ADC0-A0
- net P2-1/ADC0 renamed P2-1/ADC0-A1
- net P2-2/ADC0 renamed P2-2/ADC0-A4
- net P2-3/ADC0 renamed P2-3/ADC0-A2
- net P3-0/PWM0 renamed P3-0/PWM0-A0
- net P3-10/PWM0 renamed P3-10/PWM0-A2
- net P3-11/PWM0 renamed P3-11/PWM0-B2
- net P3-12/PWM0 renamed P3-12/PWM0-X2
- net P3-13/PWM0 renamed P3-13/PWM0-X1
- net P3-14/PWM0 renamed P3-14/PWM0-X2
- net P3-30/ADC0 renamed P3-30/ADC0-A13
- net P3-31/ADC0 renamed P3-31/ADC0-A12
- net P3-6/PWM0 renamed P3-6/PWM0-A0
- net P3-7/PWM0 renamed P3-7/PWM0-B0
- net P3-8/PWM0 renamed P3-8/PWM0-A1
- net P3-9/PWM0 renamed P3-9/PWM0-B1
- net VDD_BOARD renamed VDD-BOARD
Other:
- note removed: "A0"
- note removed: "A1"
- note removed: "A10"
- note removed: "A11"
- note removed: "A12"
- note removed: "A13"
- note removed: "A2"
- note removed: "A20"
- note removed: "A21"
- note removed: "A4"
- note removed: "A8"
- note removed: "X1"
- note removed: "X2"
- moved on the sheet: H1, H2, H3, H4, J1, J2, J3, J4
