File: tracks/A/Kicad/MCX-A153_Shield_Template.kicad_pcb (KiCad board)
At the start: 2 copper layers, 91.4 x 54.6 mm, 13 parts, among them J1 Conn_02x08_Odd_Even, J2 Conn_02x10_Odd_Even, J3 Conn_02x08_Odd_Even

Commit message: minor tweaks before 1st release.  Added Altium version
Parts:
- moved G*** 4.93 mm to (186.5, 100.1)
- renumbered JJ4 to J4
Connections:
- net /LDO_3v3 renamed /LDO-3v3
- net /MCU_Reset renamed /MCU-RESETb
- net /P1-10/ADC0 renamed /P1-10/ADC0-A8
- net /P1-12/ADC0 renamed /P1-12/ADC0-A10
- net /P1-13/ADC0 renamed /P1-13/ADC0-A11
- net /P1-4/ADC0 renamed /P1-4/ADC0-A20
- net /P1-4/RXD renamed /P1-4/UART2-RXD
- net /P1-5/ADC0 renamed /P1-5/ADC0-A21
- net /P1-5/TXD renamed /P1-5/UART2-TXD
- net /P2-0/ADC0 renamed /P2-0/ADC0-A0
- net /P2-1/ADC0 renamed /P2-1/ADC0-A1
- net /P2-2/ADC0 renamed /P2-2/ADC0-A4
- net /P2-3/ADC0 renamed /P2-3/ADC0-A2
- net /P3-0/PWM0 renamed /P3-0/PWM0-A0
- net /P3-10/PWM0 renamed /P3-10/PWM0-A2
- net /P3-11/PWM0 renamed /P3-11/PWM0-B2
- net /P3-12/PWM0 renamed /P3-12/PWM0-X2
- net /P3-13/PWM0 renamed /P3-13/PWM0-X1
- net /P3-14/PWM0 renamed /P3-14/PWM0-X2
- net /P3-30/ADC0 renamed /P3-30/ADC0-A13
- net /P3-31/ADC0 renamed /P3-31/ADC0-A12
- net /P3-6/PWM0 renamed /P3-6/PWM0-A0
- net /P3-7/PWM0 renamed /P3-7/PWM0-B0
- net /P3-8/PWM0 renamed /P3-8/PWM0-A1
- net /P3-9/PWM0 renamed /P3-9/PWM0-B1
- net /VDD_BOARD renamed /VDD-BOARD
Other:
- board text added: "2024-01-30"

Commit message: minor text fix on PCB
Other:
- board text added: "FRDM-MCXA153"
- board text removed: "FRDM MCX-A153"
